File: MT7628_USB_MODEM/MT7628_USB_MODEM.sch (KiCad schematic (older format))
At the start: 35 parts, among them J1 USB_A, J2 8P8C_LED, J3 Barrel_Jack

Commit message: update
Parts:
- removed D1, D2: MP1524, Package_SO:SOIC-8-1EP_3.9x4.9mm_P1.27mm_EP2.29x3mm_ThermalVias, symbol Library:MP1524
- removed J3: Barrel_Jack, Connector_BarrelJack:BarrelJack_Horizontal, symbol Connector:Barrel_Jack
- added C11: 1000u, Capacitor_THT:CP_Radial_D8.0mm_P2.50mm, symbol Device:CP
- added C12: 1u, Capacitor_SMD:C_0805_2012Metric, symbol Device:C
- added C13, C14: 470u, Capacitor_THT:CP_Radial_D6.3mm_P2.50mm, symbol Device:CP
- added C15, C16: 100n, Capacitor_SMD:C_0805_2012Metric, symbol Device:C
- added D1, D2: MP1584, Package_SO:SOIC-8-1EP_3.9x4.9mm_P1.27mm_EP2.29x3mm_ThermalVias, symbol MT7628_USB_MODEM-rescue:MP1584
- added D6: 1N5400, Diode_SMD:D_2512_6332Metric, symbol Diode:1N5400
- added D7: LED_Power, LED_SMD:LED_0805_2012Metric, symbol Device:LED
- added F1: Fuse, Fuse:Fuse_0805_2012Metric_Castellated, symbol Device:Fuse
- added J3: Barrel_Jack_Switch, Connector_BarrelJack:BarrelJack_Horizontal, symbol Connector:Barrel_Jack_Switch
- added J4, J5, J6: Conn_01x03_Female, Connector_PinSocket_2.54mm:PinSocket_1x03_P2.54mm_Vertical, symbol Connector:Conn_01x03_Female
- added J7: Conn_01x02_Male, Connector_PinHeader_2.54mm:PinHeader_1x02_P2.54mm_Vertical, symbol Connector:Conn_01x02_Male
- added Q1: BC817, Package_TO_SOT_SMD:SOT-23, symbol Transistor_BJT:BC817
- added R15, R16: 3k, Resistor_SMD:R_0603_1608Metric, symbol Device:R
- added R17, R25: 2k, Resistor_SMD:R_0603_1608Metric, symbol Device:R
- added R18, R19, R20, R21: 100, Resistor_SMD:R_0603_1608Metric, symbol Device:R
- added R22, R23: 1k, Resistor_SMD:R_0603_1608Metric, symbol Device:R
- added R24: 0, Resistor_SMD:R_0805_2012Metric, symbol Device:R
- added SW1: Reset, Button_Switch_SMD:SW_DIP_SPSTx01_Slide_6.7x4.1mm_W6.73mm_P2.54mm_LowProfile_JPin, symbol Switch:SW_Push
- C1, C10, C2, C9: footprint Capacitor_SMD:C_0805_2012Metric -> Capacitor_SMD:C_1206_3216Metric
- C8: value C -> n/a
- D3, D4: footprint Diode_SMD:D_0805_2012Metric -> Diode_SMD:D_1206_3216Metric
- D5: footprint RF_WiFi:HLK7628N -> Project:HLK7628N; symbol Library:HLK-7628N -> MT7628_USB_MODEM-rescue:HLK-7628N-Library
- J1: footprint Connector_USB:USB_A_Molex_67643_Horizontal -> Connector_USB:USB_A_Wuerth_61400826021_Horizontal_Stacked
- L1, L2: footprint Inductor_SMD:L_2816_7142Metric_Pad3.20x4.45mm_HandSolder -> Inductor_SMD:L_7.3x7.3_H4.5
- TR1: footprint Transformer_SMD:Transformer_Ethernet_Bourns_PT61017PEL -> Transformer_THT:TF-1016DG; symbol Library:TF-1016 -> MT7628_USB_MODEM-rescue:TF-1016-Library
Connections:
- net +3V3: now also C14.1, C16.1, R15.1, R16.1, R22.1, R23.1
- net +5V: now also C13.1
- net GND: now also J2.9, C11.2, C12.2, C13.2, C14.2, C15.2, C16.2, D1.5 (GND), D1.9 (GND), D2.5 (GND), D2.9 (GND), D6.2 (A), J4.3 (Pin_3), J5.2 (Pin_2), J6.2 (Pin_2), Q1.2 (E), R17.2, R24.2, SW1.1; no longer J1.5 (Shield)
- net Vin+: now also F1.1, J3.1; no longer C1.1, C2.1, R1.1, R4.1
- net Vin-: now also J3.2, J3.3, R24.1
- net RX1+: now reaches TR1.12 (TX+)
- net RX1+: now also J2.3; no longer J2.1
- net at J2.10: now also R23.2
- net ETH1: now reaches J2.11
- net ETH1: now also D5.12 (EPHY_LED1)
- net at J2.12: now also R22.2
- net RX1-: now reaches TR1.10 (TX-)
- net RX1-: now also J2.6; no longer J2.2
- net TX1+: now reaches TR1.9 (RX+)
- net TX1+: now also J2.1; no longer J2.3
- net TX1-: now reaches TR1.7 (RX-)
- net TX1-: now also J2.2; no longer J2.6
- net at D5.37 (MDI_TN_P0): no longer TR1.1 (TD+)
- net at D5.36 (MDI_TP_P0): no longer TR1.3 (TD-)
- net at D5.35 (MDI_RN_P0): no longer TR1.4 (RD+)
- net at D5.34 (MDI_RP_P0): no longer TR1.6 (RD-)
- net RST: now reaches D5.14 (PORST_N)
- net RST: now also C15.1, SW1.2
- net TX1: now reaches D5.15 (UART_TXD1)
- net TX1: now also R20.2
- net RX1: now reaches D5.16 (UART_RXD1)
- net RX1: now also R18.2
- net I2C_SCKL: now reaches D5.24 (I2C_SCKL)
- net I2C_SCKL: now also J4.1 (Pin_1), R16.2
- net I2C_SD: now reaches D5.25 (I2C_SD)
- net I2C_SD: now also J4.2 (Pin_2), R15.2
- net GPIO0: now reaches D5.30 (GPIO0)
- net GPIO0: now also R25.2
- net TX0: now reaches D5.31 (UART_TXD0)
- net TX0: now also R21.2
- net RX0: now reaches D5.32 (UART_RXD0)
- net RX0: now also R19.2
- net P1_T_P: now reaches D5.38 (MDI_TP_P1)
- net P1_T_P: now also TR1.6 (RD-)
- net P1_T_N: now reaches D5.39 (MDI_TN_P1)
- net P1_T_N: now also TR1.4 (RD+)
- net P1_R_P: now reaches D5.40 (MDI_RP_P1)
- net P1_R_P: now also TR1.3 (TD-)
- net P1_R_N: now reaches D5.41 (MDI_RN_P1)
- net P1_R_N: now also TR1.1 (TD+)
- net at R3.1: now also D2.6 (FREQ)
- net at C3.1, D3.1 (K), L1.1: now also D2.1 (SW)
- net at R1.2, R2.1: now also D2.2 (EN)
- net at C5.1, C7.1: now also D2.3 (COMP)
- net at R11.2, R9.1: now also D2.4 (FB)
- net at C3.2: now also D2.8 (BST)
- net at R6.1: now also D1.6 (FREQ)
- net at R4.2, R5.1: now also D1.2 (EN)
- net at C6.1, C8.1: now also D1.3 (COMP)
- net at C4.1, D4.1 (K), L2.1: now also D1.1 (SW)
- net at C4.2: now also D1.8 (BST)
- net at R10.1, R12.2: now also D1.4 (FB)
- net ETH0: no longer names the net of D5.13 (EPHY_LED0)
- new net: J6.1 (Pin_1), R19.1
- new net: J6.3 (Pin_3), R21.1
- new net: D7.1 (K), R17.1
- new net: Q1.1 (B), R25.1
- new net: J7.1 (Pin_1), Q1.3 (C)
- new net: J5.1 (Pin_1), R18.1
- new net: J5.3 (Pin_3), R20.1
- new net V+: C1.1, C11.1, C12.1, C2.1, D1.7 (VIN), D2.7 (VIN), D6.1 (K), D7.2 (A), F1.2, J7.2 (Pin_2), R1.1, R4.1
Other:
- moved on the sheet: R13, R14, TR1
